Commit message: uploaded pipeline

File: panthera_python/Panthera-HT_description/urdf/Panthera-HT_description_follower.urdf (robot description, URDF)
Before this commit: robot Panthera-HT_description, 8 links, 7 joints
Links:
- added link screen_payload, mass 3.0
Joints:
- added joint screen_payload_joint: type fixed, parent link6, child screen_payload, origin xyz=0.025 0 0 rpy=0 0 0
